File: pcb/ice_tube_clock/ice_tube_clock.brd (EAGLE design)
At the start: 148.6 x 76.2 mm, 11 parts, among them IC1 7805TV

Commit message: I thought I committed all this stuff
Parts:
- added C4, C5, C6: (no value), SparkFun-Capacitors:CAP-PTH-SMALL-KIT
- added R1, R2, R3, R4, R5, R6, R7, R8, R9: (no value), resistor:0204/7
- added U$10, U$9: PEL12S, boztalay:PEL12S
- added U$8: VFD-DRIVER-CARRIER, boztalay:VFD-DRIVER-CARRIER
- U$1: value ATMEGA168-ZIF-28 -> ATMEGA168-DIP28; device boztalay:ZIF-28 -> boztalay:DIP28
- moved U$1 204.9 mm to (124.5, 31.8)
- moved C3 195.4 mm to (106.7, 14.0), turned to 90 degrees
- moved C2 194.1 mm to (124.5, 39.4), turned to 180 degrees
- moved C1 136.1 mm to (73.0, 53.8)
- moved IC1 125.0 mm to (73.0, 63.5)
- moved U$7 102.8 mm to (73.0, 69.8), turned to 270 degrees
- moved U$6 76.2 mm to (127.0, 52.1)
- moved U$5 73.6 mm to (95.2, 52.1)
- moved U$2 63.2 mm to (10.2, 12.7), turned to 270 degrees
- moved U$4 33.1 mm to (50.8, 52.1)
- moved U$3 2.84 mm to (19.1, 52.1)
Connections:
- new net +12V: IC1.1, U$2.VCC, U$3.FIL, U$7.POS
- new net +5V: C1.1, C2.1, IC1.3, R2.2, R3.2, R6.2, R7.2, U$1.7, U$8.VCC
- new net ET: C4.1, R5.1, U$1.23
- new net GND: C1.2, C2.2, C3.1, C4.2, C5.2, C6.1, IC1.2, R1.2, U$1.22, U$1.8, U$10.C, U$2.GND, U$7.NEG, U$8.GND, U$9.C
- new net N$1: U$3.FIL_, U$4.FIL
- new net N$10: U$3.G, U$8.6
- new net N$11: U$3.H, U$8.7
- new net N$13: U$4.A, U$8.8
- new net N$14: U$4.B, U$8.9
- new net N$15: U$4.C, U$8.10
- new net N$16: U$4.D, U$8.11
- new net N$17: U$4.E, U$8.12
- new net N$18: U$4.F, U$8.13
- new net N$19: U$4.G, U$8.14
- new net N$2: U$4.FIL_, U$5.FIL
- new net N$20: U$4.H, U$8.15
- new net N$21: U$6.H, U$8.31
- new net N$22: U$6.G, U$8.30
- new net N$23: U$6.F, U$8.29
- new net N$24: U$6.E, U$8.28
- new net N$25: U$6.D, U$8.27
- new net N$26: U$6.C, U$8.26
- new net N$27: U$6.B, U$8.25
- new net N$28: U$6.A, U$8.24
- new net N$29: U$5.H, U$8.23
- new net N$3: U$5.FIL_, U$6.FIL
- new net N$30: U$5.G, U$8.22
- new net N$31: U$5.F, U$8.21
- new net N$32: U$5.E, U$8.20
- new net N$33: U$5.D, U$8.19
- new net N$34: U$5.C, U$8.18
- new net N$35: U$5.B, U$8.17
- new net N$36: U$5.A, U$8.16
- new net N$37: R1.1, U$6.FIL_
- new net N$38: U$1.15, U$8.BLANK
- new net N$39: U$1.16, U$8.LOAD
- new net N$4: U$3.A, U$8.0
- new net N$40: U$1.17, U$8.DIN
- new net N$41: U$1.18, U$8.CLK
- new net N$43: C3.2, R4.1, U$1.24
- new net N$44: R3.1, R5.2, U$10.A
- new net N$45: R6.1, R9.2, U$9.A
- new net N$46: R7.1, R8.2, U$9.B
- new net N$47: R2.1, R4.2, U$10.B
- new net N$48: C5.1, R9.1, U$1.25
- new net N$49: C6.2, R8.1, U$1.26
- new net N$5: U$3.B, U$8.1
- new net N$6: U$3.C, U$8.2
- new net N$7: U$3.D, U$8.3
- new net N$8: U$3.E, U$8.4
- new net N$9: U$3.F, U$8.5
- new net VBOOST: U$2.BST, U$3.GRID, U$4.GRID, U$5.GRID, U$6.GRID, U$8.VBB
Routing:
- net GND: track 0.00 -> 413.0 mm
- net +5V: track 0.00 -> 267.4 mm
- net VBOOST: track 0.00 -> 237.7 mm
- net +12V: track 0.00 -> 118.8 mm
- net N$41: track 0.00 -> 105.4 mm
- net N$40: track 0.00 -> 98.3 mm
- net N$39: track 0.00 -> 92.6 mm
- net N$38: track 0.00 -> 86.9 mm
- net N$21: track 0.00 -> 79.7 mm
- net N$22: track 0.00 -> 75.8 mm
- net N$4: track 0.00 -> 73.0 mm
- net N$23: track 0.00 -> 71.8 mm
- net N$5: track 0.00 -> 69.4 mm
- net N$24: track 0.00 -> 68.1 mm
- net N$6: track 0.00 -> 65.8 mm
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Other:
- board size 148.6 x 76.2 mm -> 146.1 x 80 mm
