File: pcb/ice_tube_clock/ice_tube_clock.sch (EAGLE design)
At the start: 1 part

Commit message: More big parts
Parts:
- added U$2: IV11-BOOST-SUPPLY, boztalay:IV11-BOOST-SUPPLY
- added U$3, U$4, U$5, U$6: IV-11-CARRIER, boztalay:IV-11-CARRIER
Changed lines of the file:
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@@
 <setting verticaltext="up"/>
 </settings>
-<grid distance="0.1" unitdist="inch" unit="inch" style="lines" multiple="1" display="yes" altdistance="0.01" altunitdist="inch" altunit="inch"/>
+<grid distance="0.1" unitdist="inch" unit="inch" style="lines" multiple="1" display="no" altdistance="0.01" altunitdist="inch" altunit="inch"/>
 <layers>
 <layer number="1" name="Top" color="4" fill="1" visible="no" active="no"/>
@@
 <parts>
 <part name="U$1" library="boztalay" deviceset="ATMEGA168-ZIF-28" device=""/>
+<part name="U$2" library="boztalay" deviceset="IV11-BOOST-SUPPLY" device=""/>
+<part name="U$3" library="boztalay" deviceset="IV-11-CARRIER" device=""/>
+<part name="U$4" library="boztalay" deviceset="IV-11-CARRIER" device=""/>
+<part name="U$5" library="boztalay" deviceset="IV-11-CARRIER" device=""/>
+<part name="U$6" library="boztalay" deviceset="IV-11-CARRIER" device=""/>
 </parts>
 <sheets>
@@
 <instances>
 <instance part="U$1" gate="G$1" x="-33.02" y="-7.62"/>
+<instance part="U$2" gate="G$1" x="33.02" y="-7.62"/>
+<instance part="U$3" gate="G$1" x="-68.58" y="33.02"/>
+<instance part="U$4" gate="G$1" x="-27.94" y="33.02"/>
+<instance part="U$5" gate="G$1" x="20.32" y="33.02"/>
+<instance part="U$6" gate="G$1" x="66.04" y="33.02"/>
 </instances>
 <busses>

Commit message: Starting on basic layout of the board
Parts:
- added C1: (no value), SparkFun-Passives:CAP_POLPTH1
- added C2, C3: (no value), SparkFun-Capacitors:0.1UF-50V-20%(PTH)KIT-EZ
- added IC1: 7805TV, linear:7805TV
- added U$7: PJ-037A, boztalay:PJ-037A
Changed lines of the file:
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@@
 <layer number="48" name="Document" color="7" fill="1" visible="no" active="no"/>
 <layer number="49" name="Reference" color="7" fill="1" visible="no" active="no"/>
+<layer number="50" name="dxf" color="7" fill="1" visible="no" active="no"/>
 <layer number="51" name="tDocu" color="7" fill="1" visible="no" active="no"/>
 <layer number="52" name="bDocu" color="7" fill="1" visible="no" active="no"/>
+<layer number="53" name="tGND_GNDA" color="7" fill="9" visible="no" active="no"/>
+<layer number="54" name="bGND_GNDA" color="1" fill="9" visible="no" active="no"/>
+<layer number="56" name="wert" color="7" fill="1" visible="no" active="no"/>
 <layer number="90" name="Modules" color="5" fill="1" visible="yes" active="yes"/>
 <layer number="91" name="Nets" color="2" fill="1" visible="yes" active="yes"/>
@@
 <layer number="97" name="Info" color="7" fill="1" visible="yes" active="yes"/>
 <layer number="98" name="Guide" color="6" fill="1" visible="yes" active="yes"/>
+<layer number="100" name="Muster" color="7" fill="1" visible="no" active="no"/>
+<layer number="101" name="Patch_Top" color="12" fill="4" visible="yes" active="yes"/>
+<layer number="102" name="Vscore" color="7" fill="1" visible="yes" active="yes"/>
+<layer number="103" name="tMap" color="7" fill="1" visible="yes" active="yes"/>
+<layer number="104" name="Name" color="16" fill="1" visible="yes" active="yes"/>
+<layer number="105" name="tPlate" color="7" fill="1" visible="yes" active="yes"/>
+<layer number="106" name="bPlate" color="7" fill="1" visible="yes" active="yes"/>
+<layer number="107" name="Crop" color="7" fill="1" visible="yes" active="yes"/>
+<layer number="108" name="tplace-old" color="10" fill="1" visible="yes" active="yes"/>
+<layer number="109" name="ref-old" color="11" fill="1" visible="yes" active="yes"/>
+<layer number="116" name="Patch_BOT" color="9" fill="4" visible="yes" active="yes"/>
+<layer number="121" name="_tsilk" color="7" fill="1" visible="yes" active="yes"/>
+<layer number="122" name="_bsilk" color="7" fill="1" visible="yes" active="yes"/>
+<layer number="125" name="_tNames" color="7" fill="1" visible="yes" active="yes"/>
+<layer number="144" name="Drill_legend" color="7" fill="1" visible="yes" active="yes"/>
+<layer number="151" name="HeatSink" color="7" fill="1" visible="yes" active="yes"/>
+<layer number="199" name="Contour" color="7" fill="1" visible="yes" active="yes"/>
+<layer number="200" name="200bmp" color="1" fill="10" visible="yes" active="yes"/>
+<layer number="201" name="201bmp" color="2" fill="10" visible="yes" active="yes"/>
+<layer number="202" name="202bmp" color="3" fill="10" visible="yes" active="yes"/>
+<layer number="203" name="203bmp" color="4" fill="10" visible="yes" active="yes"/>
+<layer number="204" name="204bmp" color="5" fill="10" visible="yes" active="yes"/>
+<layer number="205" name="205bmp" color="6" fill="10" visible="yes" active="yes"/>
+<layer number="206" name="206bmp" color="7" fill="10" visible="yes" active="yes"/>
+<layer number="207" name="207bmp" color="8" fill="10" visible="yes" active="yes"/>
+<layer number="208" name="208bmp" color="9" fill="10" visible="yes" active="yes"/>
+<layer number="209" name="209bmp" color="7" fill="1" visible="yes" active="yes"/>
+<layer number="210" name="210bmp" color="7" fill="1" visible="yes" active="yes"/>
+<layer number="211" name="211bmp" color="7" fill="1" visible="yes" active="yes"/>
+<layer number="212" name="212bmp" color="7" fill="1" visible="yes" active="yes"/>
+<layer number="213" name="213bmp" color="7" fill="1" visible="yes" active="yes"/>
+<layer number="214" name="214bmp" color="7" fill="1" visible="yes" active="yes"/>
+<layer number="215" name="215bmp" color="7" fill="1" visible="yes" active="yes"/>
+<layer number="216" name="216bmp" color="7" fill="1" visible="yes" active="yes"/>
+<layer number="217" name="217bmp" color="18" fill="1" visible="no" active="no"/>
+<layer number="218" name="218bmp" color="19" fill="1" visible="no" active="no"/>
+<layer number="219" name="219bmp" color="20" fill="1" visible="no" active="no"/>
+<layer number="220" name="220bmp" color="21" fill="1" visible="no" active="no"/>
+<layer number="221" name="221bmp" color="22" fill="1" visible="no" active="no"/>
+<layer number="222" name="222bmp" color="23" fill="1" visible="no" active="no"/>
+<layer number="223" name="223bmp" color="24" fill="1" visible="no" active="no"/>
+<layer number="224" name="224bmp" color="25" fill="1" visible="no" active="no"/>
+<layer number="250" name="Descript" color="3" fill="1" visible="no" active="no"/>
+<layer number="251" name="SMDround" color="12" fill="11" visible="no" active="no"/>
+<layer number="254" name="cooling" color="7" fill="1" visible="yes" active="yes"/>
 </layers>
 <schematic xreflabel="%F%N/%S.%C%R" xrefpart="/%S.%C%R">
@@
 <part name="U$5" library="boztalay" deviceset="IV-11-CARRIER" device=""/>
 <part name="U$6" library="boztalay" deviceset="IV-11-CARRIER" device=""/>
+<part name="U$7" library="boztalay" deviceset="PJ-037A" device=""/>
+<part name="IC1" library="linear" deviceset="78*" device="TV" technology="05"/>
+<part name="C1" library="SparkFun-Passives" deviceset="CAP_POL" device="PTH1"/>
+<part name="C2" library="SparkFun-Capacitors" deviceset="0.1UF-50V-20%(PTH)" device="KIT-EZ"/>
+<part name="C3" library="SparkFun-Capacitors" deviceset="0.1UF-50V-20%(PTH)" device="KIT-EZ"/>
 </parts>
 <sheets>
@@
 <instance part="U$5" gate="G$1" x="20.32" y="33.02"/>
 <instance part="U$6" gate="G$1" x="66.04" y="33.02"/>
+<instance part="U$7" gate="G$1" x="73.66" y="-7.62"/>
+<instance part="IC1" gate="A1" x="-68.58" y="-2.54"/>
+<instance part="C1" gate="G$1" x="-76.2" y="-15.24"/>
+<instance part="C2" gate="G$1" x="-7.62" y="-7.62"/>
+<instance part="C3" gate="G$1" x="-7.62" y="-17.78"/>
 </instances>
 <busses>

Commit message: I thought I committed all this stuff
Parts:
- added C4, C5, C6: (no value), SparkFun-Capacitors:0.1UF-50V-20%(PTH)KIT-EZ
- added R1, R2, R3, R4, R5, R6, R7, R8, R9: (no value), resistor:R-US_0204/7
- added U$10, U$9: PEL12S, boztalay:PEL12S
- added U$8: VFD-DRIVER-CARRIER, boztalay:VFD-DRIVER-CARRIER
- U$1: value ATMEGA168-ZIF-28 -> ATMEGA168-DIP28; device boztalay:ATMEGA168-ZIF-28 -> boztalay:ATMEGA168-DIP28
Connections:
- new net +12V: IC1.VI, U$2.VCC, U$3.FIL, U$7.POS
- new net +5V: C1.+, C2.1, IC1.VO, R2.2, R3.2, R6.2, R7.2, U$1.VCC, U$8.VCC
- new net ET: C4.1, R5.1, U$1.PC0
- new net GND: C1.-, C2.2, C3.1, C4.2, C5.2, C6.1, IC1.GND, R1.2, U$1.GND, U$1.GND_, U$10.C, U$2.GND, U$7.NEG, U$8.GND, U$9.C
- new net N$1: U$3.FIL_, U$4.FIL
- new net N$10: U$3.G, U$8.OUT6
- new net N$11: U$3.H, U$8.OUT7
- new net N$13: U$4.A, U$8.OUT8
- new net N$14: U$4.B, U$8.OUT9
- new net N$15: U$4.C, U$8.OUT10
- new net N$16: U$4.D, U$8.OUT11
- new net N$17: U$4.E, U$8.OUT12
- new net N$18: U$4.F, U$8.OUT13
- new net N$19: U$4.G, U$8.OUT14
- new net N$2: U$4.FIL_, U$5.FIL
- new net N$20: U$4.H, U$8.OUT15
- new net N$21: U$6.H, U$8.OUT31
- new net N$22: U$6.G, U$8.OUT30
- new net N$23: U$6.F, U$8.OUT29
- new net N$24: U$6.E, U$8.OUT28
- new net N$25: U$6.D, U$8.OUT27
- new net N$26: U$6.C, U$8.OUT26
- new net N$27: U$6.B, U$8.OUT25
- new net N$28: U$6.A, U$8.OUT24
- new net N$29: U$5.H, U$8.OUT23
- new net N$3: U$5.FIL_, U$6.FIL
- new net N$30: U$5.G, U$8.OUT22
- new net N$31: U$5.F, U$8.OUT21
- new net N$32: U$5.E, U$8.OUT20
- new net N$33: U$5.D, U$8.OUT19
- new net N$34: U$5.C, U$8.OUT18
- new net N$35: U$5.B, U$8.OUT17
- new net N$36: U$5.A, U$8.OUT16
- new net N$37: R1.1, U$6.FIL_
- new net N$38: U$1.PB1, U$8.BLANK
- new net N$39: U$1.PB2, U$8.LOAD
- new net N$4: U$3.A, U$8.OUT0
- new net N$40: U$1.PB3, U$8.DIN
- new net N$41: U$1.PB4, U$8.CLK
- new net N$43: C3.2, R4.1, U$1.PC1
- new net N$44: R3.1, R5.2, U$10.A
- new net N$45: R6.1, R9.2, U$9.A
- new net N$46: R7.1, R8.2, U$9.B
- new net N$47: R2.1, R4.2, U$10.B
- new net N$48: C5.1, R9.1, U$1.PC2
- new net N$49: C6.2, R8.1, U$1.PC3
- new net N$5: U$3.B, U$8.OUT1
- new net N$6: U$3.C, U$8.OUT2
- new net N$7: U$3.D, U$8.OUT3
- new net N$8: U$3.E, U$8.OUT4
- new net N$9: U$3.F, U$8.OUT5
- new net VBOOST: U$2.BST, U$3.GRID, U$4.GRID, U$5.GRID, U$6.GRID, U$8.VBB
Other:
- moved on the sheet: C1, C2, C3, IC1
